File: V1.1_Project/New_Project/EMG_FSR.brd (EAGLE design)
At the start: 20 x 50 mm, 49 parts, among them IC1 TC7660SEOA, IC2 AD8677AUJZ-REEL7, IC3 INA118U_2K5

Commit message: Located Some Parts
Parts:
- moved AMP_OUT 71.2 mm to (12.5, 1.83)
- moved HI_PASS 70.4 mm to (7.30, 2.09), turned to 180 degrees
- moved EMGOUT 61.3 mm to (4.59, 1.91)
- moved LO_PASS 57.6 mm to (9.75, 1.91)
- moved VCC- 55.8 mm to (15.2, 1.99)
- moved EMG_OUT 54.3 mm to (13.9, 47.7), turned to 180 degrees
- moved C5 53.3 mm to (3.31, 10.5), flipped to the bottom, turned to 90 degrees
- moved R20 53.3 mm to (3.57, 48.0), turned to 270 degrees
- moved IC1 51.3 mm to (10.1, 33.8)
- moved C4 48.4 mm to (3.31, 17.3), flipped to the bottom, turned to 90 degrees
- moved PAD2 48.3 mm to (17.7, 23.5), flipped to the bottom, turned to 270 degrees
- moved PAD1 44.8 mm to (17.7, 26.7), flipped to the bottom, turned to 270 degrees
- moved IC2 38.5 mm to (4.64, 25.1)
- moved VCC 34.5 mm to (6.56, 48.0)
- moved IC3 33.8 mm to (14.4, 24.8)
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
Commit message: Add files via upload
Parts:
- moved AMP_OUT 71.2 mm to (-49.5, 36.8)
- moved HI_PASS 70.4 mm to (-50.8, 41.9), turned to 0 degrees
- moved EMGOUT 61.3 mm to (-41.9, 41.9)
- moved U$3 59.6 mm to (-35.6, 3.81)
- moved LO_PASS 57.6 mm to (-31.8, 41.9)
- moved VCC- 55.8 mm to (-17.8, 47.0)
- moved EMG_OUT 54.3 mm to (-39.4, 36.8), turned to 0 degrees
- moved C5 53.3 mm to (-49.5, 3.81), flipped to the top, turned to 0 degrees
- moved R20 53.3 mm to (-49.5, 52.1), turned to 0 degrees
- moved IC1 51.3 mm to (-39.4, 20.3)
- moved C4 48.4 mm to (-43.2, 3.81), flipped to the top, turned to 0 degrees
- moved PAD2 48.3 mm to (-30.5, 20.3), flipped to the top, turned to 0 degrees
- moved PAD1 44.8 mm to (-26.7, 20.3), flipped to the top, turned to 0 degrees
- moved U$2 38.7 mm to (-27.9, 0.00)
- moved IC2 38.5 mm to (-22.9, 52.1)
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Connections:
- new net N$8: R6.2, U$1.2
- net N$19: no longer R6.2, U$1.2
Other:
- board size 20 x 50 mm -> 160 x 100 mm
