File: V1.1_Project/New_Project/EMG_FSR.brd (EAGLE design)
At the start: 20 x 50 mm, 49 parts, among them IC1 TC7660SEOA, IC2 AD8677AUJZ-REEL7, IC3 INA118U_2K5

Commit message: Add files via upload
Parts:
- removed C3: 10uF, rcl:C0402K
- removed R15, R16: 68K, rcl:R0201
- removed R18: 75K, rcl:R0201
- removed R5: 1K, rcl:R0201
- added C13: 10uF, rcl:C0805K
- added GND1: 0V, wirepad:1,6/0,8
- added R21, R24, R25: 24K, adafruit:R0402
- added R26: 68K, adafruit:R0402
- added VCC1: +5V, wirepad:1,6/0,8
- C1: value 10uF -> 10pF; device rcl:C0603K -> rcl:HPC0201
- C2: value 10pF -> 10uF; device rcl:C0402K -> rcl:C0805
- C4, C5, C8, C9: device rcl:C1206 -> rcl@1:C1206
- C6, C7: device rcl:C0805 -> rcl@1:C0805
- R1: value 16K -> 75K
- R10, R14: value 51K -> 68K; device rcl:R0201 -> adafruit:R0402
- R11: device adafruit:R0603 -> adafruit@1:R0603
- R12: device adafruit:R0603 -> adafruit@2:R0603
- R13: value 16K -> 1K; device rcl:R0201 -> adafruit:R0402
- R17: value 24K -> 68K; device rcl:R0201 -> adafruit:R0402
- R2: value 24K -> 51K
- R3: device rcl:R0805 -> rcl@1:R0805
- R4: device adafruit:R0402 -> adafruit@2:R0402
- R6: value 24K -> 51K; device rcl:R0201 -> adafruit:R0402
- R7: device adafruit:R1005 -> adafruit@2:R1005
- R8, R9: value 68K -> 16K; device rcl:R0201 -> adafruit:R0402
- moved VCC- 88.5 mm to (-55.9, 54.6)
- moved LO_PASS 88.4 mm to (-64.8, 49.5)
- moved AMP_OUT 74.3 mm to (-44.5, 49.5)
- moved VCC 72.9 mm to (-66.0, 54.6)
- moved U$1 72.1 mm to (-61.0, 5.08)
- moved GND 70.1 mm to (-61.0, 54.6), turned to 0 degrees
- moved FSR_OUT 66.0 mm to (-54.6, 49.5)
- moved HI_PASS 64.7 mm to (-30.5, 54.6), turned to 0 degrees
- moved IC1 62.2 mm to (-52.1, 33.0)
- moved PAD2 61.6 mm to (-43.2, 33.0), flipped to the top, turned to 0 degrees
- moved EMGOUT 58.8 mm to (-21.6, 54.6)
- moved PAD1 57.4 mm to (-39.4, 33.0), flipped to the top, turned to 0 degrees
- moved IC2 51.2 mm to (-33.0, 59.7)
- moved EMG_OUT 48.2 mm to (-34.3, 49.5), turned to 0 degrees
- moved IC3 46.9 mm to (-31.8, 33.0)
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Connections:
- net +5V: now also R8.2, VCC1.1; no longer R1.2
- net -5V: now also C2.1; no longer C3.1
- net EMG_BASIC: now also R25.1; no longer R17.1
- net FSR_OUT: now also R24.1; no longer R2.1
- net GND: now also GND1.1, R1.1, R2.1, R6.1; no longer R10.2, R14.1, R18.1
- net N$1: now also C13.1; no longer C1.1
- net N$10: now also R8.1; no longer R1.1
- net N$11: now also C2.2; no longer C3.2
- net N$14: now also R13.1, R21.1; no longer R5.1, R6.1
- net N$17: now also R17.2; no longer R16.2
- net N$18: now also R13.2; no longer R5.2
- net N$19: now also R2.2, R21.2; no longer R10.1, R6.2
- net N$2: now also C13.2; no longer C1.2
- net N$20: now also R14.2; no longer R9.1
- net N$21: now also R10.1, R14.1; no longer R8.1, R9.2
- net N$26: now also R6.2, R9.2; no longer R13.2, R14.2
- net N$27: now also R17.1, R26.2; no longer R15.1, R16.1
- net N$28: now also R26.1; no longer R15.2
- net N$3: now also C1.1; no longer C2.1
- net N$30: now also R1.2, R25.2; no longer R17.2, R18.2
- net N$5: now also C1.2; no longer C2.2
- net N$7: now also R24.2; no longer R2.2
- net PIN7: now also R10.2, R9.1; no longer R13.1, R8.2
Other:
- board size 20 x 50 mm -> 160 x 100 mm
