File: V1.1_Project/New_Project/EMG_FSR.sch (EAGLE design)
At the start: 49 parts, among them IC1 TC7660SEOA, IC2 AD8677AUJZ-REEL7, IC3 INA118U_2K5

Commit message: Add files via upload
Connections:
- new net N$8: R6.2, U$1.1IN-
- net N$19: no longer R6.2, U$1.1IN-
Changed lines of the file:
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@@
 <net name="N$19" class="0">
 <segment>
-<pinref part="R6" gate="G$1" pin="2"/>
-<pinref part="U$1" gate="G$1" pin="1IN-"/>
-<wire x1="-20.32" y1="-50.8" x2="-12.7" y2="-50.8" width="0.1524" layer="91"/>
 <pinref part="R10" gate="G$1" pin="1"/>
-<wire x1="-12.7" y1="-50.8" x2="-12.7" y2="-43.18" width="0.1524" layer="91"/>
-<wire x1="-12.7" y1="-43.18" x2="-45.72" y2="-43.18" width="0.1524" layer="91"/>
-<junction x="-12.7" y="-50.8"/>
+<wire x1="-17.78" y1="-43.18" x2="-45.72" y2="-43.18" width="0.1524" layer="91"/>
+<junction x="-17.78" y="-50.8"/>
+<wire x1="-17.78" y1="-43.18" x2="-17.78" y2="-50.8" width="0.1524" layer="91"/>
 </segment>
 </net>
@@
 </segment>
 </net>
+<net name="N$8" class="0">
+<segment>
+<pinref part="U$1" gate="G$1" pin="1IN-"/>
+<pinref part="R6" gate="G$1" pin="2"/>
+<wire x1="-20.32" y1="-50.8" x2="-12.7" y2="-50.8" width="0.1524" layer="91"/>
+</segment>
+</net>
