File: V1.1_Project/New_Project/IMU.sch (EAGLE design)
At the start: 46 parts, among them IC1 TC7660SEOA, IC2 AD8677AUJZ-REEL7, IC3 INA118U_2K5, U1 AZ1117EH-3.3TRG1

Commit message: Add files via upload
Parts:
- removed OUT1, OUT2, OUT3, OUT4: (no value), wirepad:1,6/0,8
- removed VIN+, VIN-: WIREPADSMD2,54-5,08, wirepad:WIREPADSMD2,54-5,08
- added AMP_OUT, EMG_OUT, HI_PASS, LO_PASS, PAD3, SCL, SDA: (no value), wirepad:1,6/0,8
- added C10, C11: 1uF, rcl:C-EUC0402
- added ORANGE, R20, RED: RESC0402X40N, RESC0402X40N:RESC0402X40N
- added R19, R22, R23: ERJ-2RKF1500X, ERJ-2RKF1500X:ERJ-2RKF1500X
- added U$2, U$3: EMG_VIA, EMG_VIA:EMG_VIA
- added U$4: IMU, IMU:IMU
Connections:
- net EMGOUT renamed RAWEMG
- new net +3.3V: C10.1, PAD3.P, R23.2, U$4.VCC, U1.OUT
- new net N$16: SDA.P, U$4.SDA
- new net N$4: R22.1, RED.1
- new net N$5: C2.2, IC3.V+IN, U$3.1
- new net N$6: R19.1, R20.1
- new net N$9: ORANGE.1, R23.1
- new net PIN7: HI_PASS.P, R12.1, R13.1, R8.2, U$1.2OUT
- net +5V: now also C11.1, R22.2, U1.IN
- net -5V: now also R20.2
- net EMG_BASIC: now also EMG_OUT.P; no longer OUT3.P
- net GND: now also C10.2, C11.2, C5.1, ORANGE.2, R10.2, R11.1, R14.1, R19.2, RED.2, U$4.GND, U1.ADJ/GND; no longer OUT2.P, R12.1, R13.1, R8.2, U$1.2OUT
- net N$14: now also LO_PASS.P; no longer OUT1.P
- net N$17: now also AMP_OUT.P; no longer OUT4.P
- net N$19: no longer R6.2, U$1.1IN-
- net N$22: now also SCL.P, U$4.SCL; no longer C5.1, R10.2, R11.1, R14.1
- net N$3: now also U$2.1; no longer VIN+.P
- net N$8: now also R6.2, U$1.1IN-; no longer C2.2, IC3.V+IN, VIN-.P
Other:
- note added: "IMU"
- moved on the sheet: C1, C2, C3, C4, C5, C6, C7, C8, C9, EMGOUT, EMG_BASIC, FSR_OUT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
