File: V1.1_Project/New_Project/IMU.sch (EAGLE design)
At the start: 46 parts, among them IC1 TC7660SEOA, IC2 AD8677AUJZ-REEL7, IC3 INA118U_2K5, U1 AZ1117EH-3.3TRG1

Commit message: Add files via upload
finished IMU layout including silkscreen
Parts:
- removed C3: 10uF, rcl:C-EUC0402K
- removed EMGOUT, EMG_BASIC, OUT1, OUT2, OUT3, OUT4: (no value), wirepad:1,6/0,8
- removed R15, R16: 68K, rcl:R-US_R0201
- removed R18: 75K, rcl:R-US_R0201
- removed R5: 1K, rcl:R-US_R0201
- removed VIN+, VIN-: WIREPADSMD2,54-5,08, wirepad:WIREPADSMD2,54-5,08
- added +3.3V, AMP_OUT, EMG_OUT, HI_PASS, LO_PASS, RAWEMG, SCL, SDA: (no value), wirepad:1,6/0,8
- added BLUE, ORANGE, RED: RESC0402X40N, RESC0402X40N:RESC0402X40N
- added C10, C11: 1uF, rcl:C-EUC0402
- added C13: 10uF, rcl:C-EUC0805K
- added GND1: 0V, wirepad:1,6/0,8
- added IMU: IMU, IMU:IMU
- added R19, R22, R23: ERJ-2RKF1500X, ERJ-2RKF1500X:ERJ-2RKF1500X
- added R21, R24, R25: 24K, adafruit:R-US_R0402
- added R26: 68K, adafruit:R-US_R0402
- added U$2, U$3: EMG_VIA, EMG_VIA:EMG_VIA
- added VCC1: +5V, wirepad:1,6/0,8
- C1: value 10uF -> 10pF; device rcl:C-EUC0603K -> rcl:C-EUHPC0201
- C2: value 10pF -> 10uF; device rcl:C-EUC0402K -> rcl:C-EUC0805
- R1: value 16K -> 75K
- R10, R14: value 51K -> 68K; device rcl:R-US_R0201 -> adafruit:R-US_R0402
- R13: value 16K -> 1K; device rcl:R-US_R0201 -> adafruit:R-US_R0402
- R17: value 24K -> 68K; device rcl:R-US_R0201 -> adafruit:R-US_R0402
- R2: value 24K -> 51K
- R6: value 24K -> 51K; device rcl:R-US_R0201 -> adafruit:R-US_R0402
- R8, R9: value 68K -> 16K; device rcl:R-US_R0201 -> adafruit:R-US_R0402
Connections:
- removed net EMGOUT: C7.1, EMGOUT.P, IC3.VO
- removed net N$8: C2.2, IC3.V+IN, VIN-.P
- new net +3.3V: +3.3V.P, C10.1, IMU.VCC, R23.2, U1.OUT
- new net N$16: IMU.SDA, SDA.P
- new net N$4: R22.1, RED.1
- new net N$5: C1.2, IC3.V+IN, U$3.1
- new net N$6: BLUE.1, R19.1
- new net N$9: ORANGE.1, R23.1
- new net PIN7: HI_PASS.P, R10.2, R12.1, R9.1, U$1.2OUT
- new net RAWEMG: C7.1, IC3.VO, RAWEMG.P
- net +5V: now also C11.1, R22.2, R8.2, U1.IN, VCC1.P; no longer R1.2
- net -5V: now also BLUE.2, C2.1; no longer C3.1
- net EMG_BASIC: now also EMG_OUT.P, R25.1; no longer EMG_BASIC.P, OUT3.P, R17.1
- net FSR_OUT: now also R24.1; no longer R2.1
- net GND: now also C10.2, C11.2, C5.1, GND1.P, IMU.GND, ORANGE.2, R1.1, R11.1, R19.2, R2.1, R6.1, RED.2, U1.ADJ/GND; no longer OUT2.P, R12.1, R13.1, R18.1, R8.2, U$1.2OUT
- net N$1: now also C13.1; no longer C1.1
- net N$10: now also R8.1; no longer R1.1
- net N$11: now also C2.2; no longer C3.2
- net N$14: now also LO_PASS.P, R13.1, R21.1; no longer OUT1.P, R5.1, R6.1
- net N$17: now also AMP_OUT.P, R17.2; no longer OUT4.P, R16.2
- net N$18: now also R13.2; no longer R5.2
- net N$19: now also R2.2, R21.2; no longer R10.1, R6.2
- net N$2: now also C13.2; no longer C1.2
- net N$20: now also R14.2; no longer R9.1
- net N$21: now also R10.1, R14.1; no longer R8.1, R9.2
- net N$22: now also IMU.SCL, SCL.P; no longer C5.1, R10.2, R11.1, R14.1
- net N$26: now also R6.2, R9.2; no longer R13.2, R14.2
- net N$27: now also R17.1, R26.2; no longer R15.1, R16.1
- net N$28: now also R26.1; no longer R15.2
- net N$3: now also C1.1, U$2.1; no longer C2.1, VIN+.P
- net N$30: now also R1.2, R25.2; no longer R17.2, R18.2
- net N$7: now also R24.2; no longer R2.2
Other:
- note added: "IMU"
- moved on the sheet: C1, C2, C4, C5, C6, C7, C8, C9, FSR_OUT, GND, IC1, IC2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
