File: V1.1_Project/New_Project/IMU.brd (EAGLE design)
At the start: 160 x 100 mm, 60 parts, among them IC1 TC7660SEOA, IC2 AD8677AUJZ-REEL7, IC3 INA118U_2K5, U1 AZ1117EH-3.3TRG1

Commit message: Add files via upload
Parts:
- C4, C5, C8, C9: device rcl@1:C1206 -> rcl:C1206
- C6, C7: device rcl@1:C0805 -> rcl:C0805
- PAD3, SCL, SDA: device wirepad@1:1,6/0,8 -> wirepad:1,6/0,8
- R11: device adafruit@1:R0603 -> adafruit:R0603
- R12: device adafruit@2:R0603 -> adafruit@1:R0603
- R3: device rcl@1:R0805 -> rcl:R0805
- R4: device adafruit@2:R0402 -> adafruit@1:R0402
- R7: device adafruit@2:R1005 -> adafruit@1:R1005
